File: e-tinkers-esp32-c3.kicad_pcb (KiCad board)
At the start: 2 copper layers, 22 x 42 mm, 22 parts, among them J1 Conn_01x10_Male, J2 Conn_01x10_Male, J3 Conn_01x04_Male, SW1 RESET, SW2 FLASH, U1 AP2112K-3.3, U2 WS2812C-2020, U3 ESP32-C3-WROOM-02

Commit message: update to kicad 6
Other:
- net class Default removed
